Commit message: Rename origin_v10_description to origin_one_description

File: origin_one_description/urdf/origin_one.urdf (robot description, URDF)
Before this commit: robot avular_origin_v10, 11 links, 10 joints
Links:
- added link imu_link
- added link us_center_front_link
- added link us_center_rear_link
- added link us_left_front_link
- added link us_left_rear_link
- added link us_right_front_link
- added link us_right_rear_link
- link gnss_link: geometry visual mesh filename=package://origin_one_description/urdf/meshes/antenna.obj scale=0.001 0.001 0.001
- link left_front_wheel: geometry collision cylinder length=.07 radius=.1175; visual mesh filename=package://origin_one_description/urdf/meshes/wheel.obj scale=0.001 0.001 0.001
- link left_rear_wheel: geometry collision cylinder length=.07 radius=.1175; visual mesh filename=package://origin_one_description/urdf/meshes/wheel.obj scale=0.001 0.001 0.001
- link main_body: geometry collision box size=.65 .4 .125; visual mesh filename=package://origin_one_description/urdf/meshes/body.obj scale=0.001 0.001 0.001
- link ouster_base: geometry collision box size=0.1 0.1 0.1; visual mesh filename=package://origin_one_description/urdf/meshes/ouster.obj scale=0.001 0.001 0.001
- link right_front_wheel: geometry collision cylinder length=.07 radius=.1175; visual mesh filename=package://origin_one_description/urdf/meshes/wheel.obj scale=0.001 0.001 0.001
- link right_rear_wheel: geometry collision cylinder length=.07 radius=.1175; visual mesh filename=package://origin_one_description/urdf/meshes/wheel.obj scale=0.001 0.001 0.001
Joints:
- added joint imu_joint: type fixed, parent main_body, child imu_link, origin xyz=-0.1266 0.0749 0.066 rpy=0 0 2.357
- added joint us_center_front_joint: type fixed, parent main_body, child us_center_front_link, origin xyz=0.322 0 0.063 rpy=0 0 0
- added joint us_center_rear_joint: type fixed, parent main_body, child us_center_rear_link, origin xyz=-0.322 0 0.063 rpy=0 0 0
- added joint us_left_front_joint: type fixed, parent main_body, child us_left_front_link, origin xyz=0.314 0.119 0.072 rpy=0 0 -0.7854
- added joint us_left_rear_joint: type fixed, parent main_body, child us_left_rear_link, origin xyz=-0.314 0.119 0.072 rpy=0 0 -2.357
- added joint us_right_front_joint: type fixed, parent main_body, child us_right_front_link, origin xyz=0.314 -0.119 0.072 rpy=0 0 0.7854
- added joint us_right_rear_joint: type fixed, parent main_body, child us_right_rear_link, origin xyz=-0.314 -0.119 0.072 rpy=0 0 2.357
- joint realsense_joint: origin xyz=0.32 0.03 0.1 rpy=0 0 0 -> xyz=0.3156 0.017 0.096 rpy=0 0 0
