Commit message: Update description package. This commit is auto-generated by the CI.

File: origin_one_description/urdf/origin_one.urdf.xacro (robot description, xacro)
@@ -1,4 +1,26 @@
 <?xml version='1.0'?>
-<robot name="avular_origin_one">
+<robot name="avular_origin_one" xmlns:xacro="http://ros.org/wiki/xacro" xmlns:ignition="http://sdformat.org/schemas/root.xsd">
+  <xacro:arg name="drive_configuration" default="skid_steer_drive"/>
+  <xacro:property name="var" value="$(arg drive_configuration)"/>
+  <xacro:if value="${var == 'skid_steer_drive'}">
+    <xacro:property name="trackWidth" value="0.500"/>
+    <xacro:property name="wheelbase" value="0.410"/>
+    <xacro:property name="wheelRadius" value="0.120"/>
+    <xacro:property name="groundClearance" value="0.064"/>
+    <!-- wheelMeshFileA refer to the mesh file used to visualize front left & rear right wheel  -->
+    <xacro:property name="wheelMeshFileA" value="package://origin_one_description/urdf/meshes/wheel.obj"/>
+    <!-- wheelMeshFileB refer to the mesh file used to visualize front right & rear left wheel  -->
+    <xacro:property name="wheelMeshFileB" value="package://origin_one_description/urdf/meshes/wheel.obj"/>
+  </xacro:if>
+  <xacro:if value="${var == 'mecanum_drive'}">
+    <xacro:property name="trackWidth" value="0.475"/>
+    <xacro:property name="wheelbase" value="0.410"/>
+    <xacro:property name="wheelRadius" value="0.1015"/>
+    <xacro:property name="groundClearance" value="0.0455"/>
+    <!-- wheelMeshFileA refer to the mesh file used to visualize front left & rear right wheel  -->
+    <xacro:property name="wheelMeshFileA" value="package://origin_one_description/urdf/meshes/wheel_mecanumA.obj"/>
+    <!-- wheelMeshFileB refer to the mesh file used to visualize front right & rear left wheel  -->
+    <xacro:property name="wheelMeshFileB" value="package://origin_one_description/urdf/meshes/wheel_mecanumB.obj"/>
+  </xacro:if>
   <gazebo>
     <static>false</static>
@@ -37,5 +59,5 @@
       <origin xyz="0 0 0.0" rpy="0 0 0"/>
       <geometry>
-        <cylinder length=".07" radius=".1175"/>
+        <cylinder length=".07" radius="${wheelRadius}"/>
       </geometry>
     </collision>
@@ -43,5 +65,5 @@
       <origin xyz="0.0 0.0 0.0" rpy="0.0 1.5707 0.0"/>
       <geometry>
-        <mesh filename="package://origin_one_description/urdf/meshes/wheel.obj"
+        <mesh filename="${wheelMeshFileA}"
           scale="0.001 0.001 0.001" />
       </geometry>
@@ -52,11 +74,20 @@
       <surface>
         <friction>
-          <ode>
-            <mu>1</mu>
-            <mu2>1</mu2>
-            <slip1>0.015</slip1>
-            <slip2>0</slip2>
-            <fdir1>0 0 1</fdir1>
-          </ode>
+          <xacro:if value="${var == 'skid_steer_drive'}">
+            <ode>
+              <mu>1</mu>
+              <mu2>1</mu2>
+              <slip1>0.015</slip1>
+              <slip2>0</slip2>
+              <fdir1>0 0 1</fdir1>
+            </ode>
+          </xacro:if>
+          <xacro:if value="${var == 'mecanum_drive'}">
+            <ode>
+              <mu>1</mu>
+              <mu2>0</mu2>
+              <fdir1 ignition:expressed_in="base_link">1 -1 0</fdir1>
+            </ode>
+          </xacro:if>
           <bullet>
             <friction>1</friction>
@@ -76,11 +107,11 @@
       <origin xyz="0 0 0.0" rpy="0 0 0"/>
       <geometry>
-        <cylinder length=".07" radius=".1175"/>
+        <cylinder length=".07" radius="${wheelRadius}"/>
       </geometry>
     </collision>
     <visual>
-      <origin xyz="0.0 0.0 0.0" rpy="0.0 1.5707 0.0"/>
-      <geometry>
-        <mesh filename="package://origin_one_description/urdf/meshes/wheel.obj"
+      <origin xyz="0.0 0.0 0.0" rpy="0.0 -1.5707 0.0"/>
+      <geometry>
+        <mesh filename="${wheelMeshFileB}"
           scale="0.001 0.001 0.001" />
       </geometry>
@@ -91,11 +122,20 @@
       <surface>
         <friction>
-          <ode>
-            <mu>1</mu>
-            <mu2>1</mu2>
-            <slip1>0.015</slip1>
-            <slip2>0</slip2>
-            <fdir1>0 0 1</fdir1>
-          </ode>
+          <xacro:if value="${var == 'skid_steer_drive'}">
+            <ode>
+              <mu>1</mu>
+              <mu2>1</mu2>
+              <slip1>0.015</slip1>
+              <slip2>0</slip2>
+              <fdir1>0 0 1</fdir1>
+            </ode>
+          </xacro:if>
+          <xacro:if value="${var == 'mecanum_drive'}">
+            <ode>
+              <mu>1</mu>
+              <mu2>0</mu2>
+              <fdir1 ignition:expressed_in="base_link">1 1 0</fdir1>
+            </ode>
+          </xacro:if>
           <bullet>
             <friction>1</friction>
@@ -115,5 +155,5 @@
       <origin xyz="0 0 0.0" rpy="0 0 0"/>
       <geometry>
-        <cylinder length=".07" radius=".1175"/>
+        <cylinder length=".07" radius="${wheelRadius}"/>
       </geometry>
     </collision>
@@ -121,5 +161,5 @@
       <origin xyz="0.0 0.0 0.0" rpy="0.0 1.5707 0.0"/>
       <geometry>
-        <mesh filename="package://origin_one_description/urdf/meshes/wheel.obj"
+        <mesh filename="${wheelMeshFileB}"
           scale="0.001 0.001 0.001" />
       </geometry>
@@ -130,11 +170,20 @@
       <surface>
         <friction>
-          <ode>
-            <mu>1</mu>
-            <mu2>1</mu2>
-            <slip1>0.015</slip1>
-            <slip2>0</slip2>
-            <fdir1>0 0 1</fdir1>
-          </ode>
+          <xacro:if value="${var == 'skid_steer_drive'}">
+            <ode>
+              <mu>1</mu>
+              <mu2>1</mu2>
+              <slip1>0.015</slip1>
+              <slip2>0</slip2>
+              <fdir1>0 0 1</fdir1>
+            </ode>
+          </xacro:if>
+          <xacro:if value="${var == 'mecanum_drive'}">
+            <ode>
+              <mu>1</mu>
+              <mu2>0</mu2>
+              <fdir1 ignition:expressed_in="base_link">1 1 0</fdir1>
+            </ode>
+          </xacro:if>
           <bullet>
             <friction>1</friction>
@@ -154,11 +203,11 @@
       <origin xyz="0 0 0.0" rpy="0 0 0"/>
       <geometry>
-        <cylinder length=".07" radius=".1175"/>
+        <cylinder length=".07" radius="${wheelRadius}"/>
       </geometry>
     </collision>
     <visual>
-      <origin xyz="0.0 0.0 0.0" rpy="0.0 1.5707 0.0"/>
-      <geometry>
-        <mesh filename="package://origin_one_description/urdf/meshes/wheel.obj"
+      <origin xyz="0.0 0.0 0.0" rpy="0.0 -1.5707 0.0"/>
+      <geometry>
+        <mesh filename="${wheelMeshFileA}"
           scale="0.001 0.001 0.001" />
       </geometry>
@@ -169,11 +218,20 @@
       <surface>
         <friction>
-          <ode>
-            <mu>1</mu>
-            <mu2>1</mu2>
-            <slip1>0.015</slip1>
-            <slip2>0</slip2>
-            <fdir1>0 0 1</fdir1>
-          </ode>
+          <xacro:if value="${var == 'skid_steer_drive'}">
+            <ode>
+              <mu>1</mu>
+              <mu2>1</mu2>
+              <slip1>0.015</slip1>
+              <slip2>0</slip2>
+              <fdir1>0 0 1</fdir1>
+            </ode>
+          </xacro:if>
+          <xacro:if value="${var == 'mecanum_drive'}">
+            <ode>
+              <mu>1</mu>
+              <mu2>0</mu2>
+              <fdir1 ignition:expressed_in="base_link">1 -1 0</fdir1>
+            </ode>
+          </xacro:if>
           <bullet>
             <friction>1</friction>
@@ -365,10 +423,10 @@
   </link>
   <joint type="fixed" name="base_body">
-    <origin xyz="0.0 0 0.064" rpy="0 0 0"/>
+    <origin xyz="0.0 0 ${groundClearance}" rpy="0 0 0"/>
     <child link="main_body" />
     <parent link="base_link"/>
   </joint>
   <joint type="continuous" name="main_body_left_front_wheel">
-    <origin xyz="0.205 0.25 0.056" rpy="-1.5707 0 0"/>
+    <origin xyz="${wheelbase/2} ${trackWidth/2} 0.056" rpy="-1.5707 0 0"/>
     <child link="left_front_wheel" />
     <parent link="main_body"/>
@@ -377,22 +435,22 @@
   </joint>
   <joint type="continuous" name="main_body_right_front_wheel">
-    <origin xyz="0.205 -0.25 0.056" rpy="1.5707 0 0"/>
+    <origin xyz="${wheelbase/2} ${-trackWidth/2} 0.056" rpy="-1.5707 0 0"/>
     <child link="right_front_wheel" />
-    <parent link="main_body"/>
-    <axis xyz="0 0 -1"/>
-    <limit effort="100000.0" velocity="10"/>
-  </joint>
-  <joint type="continuous" name="main_body_left_rear_wheel">
-    <origin xyz="-0.205 0.25 0.056" rpy="-1.5707 0 0"/>
-    <child link="left_rear_wheel" />
     <parent link="main_body"/>
     <axis xyz="0 0 1"/>
     <limit effort="100000.0" velocity="10"/>
   </joint>
+  <joint type="continuous" name="main_body_left_rear_wheel">
+    <origin xyz="${-wheelbase/2} ${trackWidth/2} 0.056" rpy="-1.5707 0 0"/>
+    <child link="left_rear_wheel" />
+    <parent link="main_body"/>
+    <axis xyz="0 0 1"/>
+    <limit effort="100000.0" velocity="10"/>
+  </joint>
   <joint type="continuous" name="main_body_right_rear_wheel">
-    <origin xyz="-0.205 -0.25 0.056" rpy="1.5707 0 0"/>
+    <origin xyz="${-wheelbase/2} ${-trackWidth/2} 0.056" rpy="-1.5707 0 0"/>
     <child link="right_rear_wheel" />
     <parent link="main_body"/>
-    <axis xyz="0 0 -1"/>
+    <axis xyz="0 0 1"/>
     <limit effort="100000.0" velocity="10"/>
   </joint>
@@ -457,30 +515,57 @@
     <parent link="main_body"/>
   </joint>
-  <!-- Controls the differential drive robot -->
   <gazebo>
     <plugin filename="gz-sim-joint-state-publisher-system" name="ignition::gazebo::systems::JointStatePublisher">
       <topic>/robot/joint_states</topic>
     </plugin>
-    <plugin filename="gz-sim-diff-drive-system" name="gz::sim::systems::DiffDrive">
-      <left_joint>main_body_left_front_wheel</left_joint>
-      <left_joint>main_body_left_rear_wheel</left_joint>
-      <right_joint>main_body_right_front_wheel</right_joint>
-      <right_joint>main_body_right_rear_wheel</right_joint>
-      <wheel_separation>0.45</wheel_separation>
-      <wheel_radius>0.120</wheel_radius>
-      <max_linear_acceleration>5.5</max_linear_acceleration>
-      <min_linear_acceleration>-5.5</min_linear_acceleration>
-      <max_angular_acceleration>6</max_angular_acceleration>
-      <min_angular_acceleration>-6</min_angular_acceleration>
-      <max_linear_velocity>1.5</max_linear_velocity>
-      <min_linear_velocity>-1.5</min_linear_velocity>
-      <max_angular_velocity>2</max_angular_velocity>
-      <min_angular_velocity>-2</min_angular_velocity>
-      <topic>/robot/cmd_vel</topic>
-      <odom_topic>/robot/odom</odom_topic>
-      <tf_topic>/robot/tf</tf_topic>
-      <frame_id>odom</frame_id>
-      <child_frame_id>base_link</child_frame_id>
-    </plugin>
+    <!-- Controls the differential drive robot -->
+    <xacro:if value="${var == 'skid_steer_drive'}">
+      <plugin filename="gz-sim-diff-drive-system" name="gz::sim::systems::DiffDrive">
+        <left_joint>main_body_left_front_wheel</left_joint>
+        <left_joint>main_body_left_rear_wheel</left_joint>
+        <right_joint>main_body_right_front_wheel</right_joint>
+        <right_joint>main_body_right_rear_wheel</right_joint>
+        <wheel_separation>0.45</wheel_separation>
+        <wheel_radius>0.120</wheel_radius>
+        <max_linear_acceleration>5.5</max_linear_acceleration>
+        <min_linear_acceleration>-5.5</min_linear_acceleration>
+        <max_angular_acceleration>6</max_angular_acceleration>
+        <min_angular_acceleration>-6</min_angular_acceleration>
+        <max_linear_velocity>1.5</max_linear_velocity>
+        <min_linear_velocity>-1.5</min_linear_velocity>
+        <max_angular_velocity>2</max_angular_velocity>
+        <min_angular_velocity>-2</min_angular_velocity>
+        <topic>/robot/cmd_vel</topic>
+        <odom_topic>/robot/odom</odom_topic>
+        <tf_topic>/robot/tf</tf_topic>
+        <frame_id>odom</frame_id>
+        <child_frame_id>base_link</child_frame_id>
+      </plugin>
+    </xacro:if>
+    <!-- Controls the mecanum drive robot -->
+    <xacro:if value="${var == 'mecanum_drive'}">
+      <plugin
+        filename="gz-sim-mecanum-drive-system" name="ignition::gazebo::systems::MecanumDrive">
+        <front_left_joint>main_body_left_front_wheel</front_left_joint>
+        <front_right_joint>main_body_right_front_wheel</front_right_joint>
+        <back_left_joint>main_body_left_rear_wheel</back_left_joint>
+        <back_right_joint>main_body_right_rear_wheel</back_right_joint>
+        <wheel_separation>${trackWidth}</wheel_separation>
+        <wheelbase>${wheelbase}</wheelbase>
+        <wheel_radius>${wheelRadius}</wheel_radius>
+        <min_acceleration>-5</min_acceleration>
+        <max_acceleration>5</max_acceleration>
+        <topic>/robot/cmd_vel</topic>
+      </plugin>
+    <!-- Seperate plugin for odometry is used because mecanum drive plug does not have this feature-->
+    <!-- see https://github.com/gazebosim/gz-sim/pull/2297 for more information -->
+      <plugin
+        filename="gz-sim-odometry-publisher-system" name="ignition::gazebo::systems::OdometryPublisher">
+        <odom_topic>/robot/odom</odom_topic>
+        <tf_topic>/robot/tf</tf_topic>
+        <odom_frame>odom</odom_frame>
+        <robot_base_frame>base_link</robot_base_frame>
+      </plugin>
+    </xacro:if>
   </gazebo>
 </robot>

Commit message: Update description package. This commit is auto-generated by the CI.

File: origin_one_description/urdf/origin_one.urdf.xacro (robot description, xacro)
@@ -12,4 +12,24 @@
     <!-- wheelMeshFileB refer to the mesh file used to visualize front right & rear left wheel  -->
     <xacro:property name="wheelMeshFileB" value="package://origin_one_description/urdf/meshes/wheel.obj"/>
+  </xacro:if>
+  <xacro:if value="${var == 'big_skid_steer_drive'}">
+    <xacro:property name="trackWidth" value="0.530"/>
+    <xacro:property name="wheelbase" value="0.410"/>
+    <xacro:property name="wheelRadius" value="0.165"/>
+    <xacro:property name="groundClearance" value="0.109"/>
+    <!-- wheelMeshFileA refer to the mesh file used to visualize front left & rear right wheel  -->
+    <xacro:property name="wheelMeshFileA" value="package://origin_one_description/urdf/meshes/wheel_big.obj"/>
+    <!-- wheelMeshFileB refer to the mesh file used to visualize front right & rear left wheel  -->
+    <xacro:property name="wheelMeshFileB" value="package://origin_one_description/urdf/meshes/wheel_big.obj"/>
+  </xacro:if>
+  <xacro:if value="${var == 'elevated_skid_steer_drive'}">
+    <xacro:property name="trackWidth" value="0.530"/>
+    <xacro:property name="wheelbase" value="0.410"/>
+    <xacro:property name="wheelRadius" value="0.165"/>
+    <xacro:property name="groundClearance" value="0.109"/>
+    <!-- wheelMeshFileA refer to the mesh file used to visualize front left & rear right wheel  -->
+    <xacro:property name="wheelMeshFileA" value="package://origin_one_description/urdf/meshes/wheel_big.obj"/>
+    <!-- wheelMeshFileB refer to the mesh file used to visualize front right & rear left wheel  -->
+    <xacro:property name="wheelMeshFileB" value="package://origin_one_description/urdf/meshes/wheel_big.obj"/>
   </xacro:if>
   <xacro:if value="${var == 'mecanum_drive'}">
@@ -90,4 +110,22 @@
             </ode>
           </xacro:if>
+          <xacro:if value="${var == 'big_skid_steer_drive'}">
+            <ode>
+              <mu>1</mu>
+              <mu2>1</mu2>
+              <slip1>0.015</slip1>
+              <slip2>0</slip2>
+              <fdir1>0 0 1</fdir1>
+            </ode>
+          </xacro:if>
+          <xacro:if value="${var == 'elevated_skid_steer_drive'}">
+            <ode>
+              <mu>1</mu>
+              <mu2>1</mu2>
+              <slip1>0.015</slip1>
+              <slip2>0</slip2>
+              <fdir1>0 0 1</fdir1>
+            </ode>
+          </xacro:if>
           <bullet>
             <friction>1</friction>
@@ -138,4 +176,22 @@
             </ode>
           </xacro:if>
+          <xacro:if value="${var == 'big_skid_steer_drive'}">
+            <ode>
+              <mu>1</mu>
+              <mu2>1</mu2>
+              <slip1>0.015</slip1>
+              <slip2>0</slip2>
+              <fdir1>0 0 1</fdir1>
+            </ode>
+          </xacro:if>
+          <xacro:if value="${var == 'elevated_skid_steer_drive'}">
+            <ode>
+              <mu>1</mu>
+              <mu2>1</mu2>
+              <slip1>0.015</slip1>
+              <slip2>0</slip2>
+              <fdir1>0 0 1</fdir1>
+            </ode>
+          </xacro:if>
           <bullet>
             <friction>1</friction>
@@ -186,4 +242,22 @@
             </ode>
           </xacro:if>
+          <xacro:if value="${var == 'big_skid_steer_drive'}">
+            <ode>
+              <mu>1</mu>
+              <mu2>1</mu2>
+              <slip1>0.015</slip1>
+              <slip2>0</slip2>
+              <fdir1>0 0 1</fdir1>
+            </ode>
+          </xacro:if>
+          <xacro:if value="${var == 'elevated_skid_steer_drive'}">
+            <ode>
+              <mu>1</mu>
+              <mu2>1</mu2>
+              <slip1>0.015</slip1>
+              <slip2>0</slip2>
+              <fdir1>0 0 1</fdir1>
+            </ode>
+          </xacro:if>
           <bullet>
             <friction>1</friction>
@@ -232,4 +306,22 @@
               <mu2>0</mu2>
               <fdir1 ignition:expressed_in="base_link">1 -1 0</fdir1>
+            </ode>
+          </xacro:if>
+          <xacro:if value="${var == 'big_skid_steer_drive'}">
+            <ode>
+              <mu>1</mu>
+              <mu2>1</mu2>
+              <slip1>0.015</slip1>
+              <slip2>0</slip2>
+              <fdir1>0 0 1</fdir1>
+            </ode>
+          </xacro:if>
+          <xacro:if value="${var == 'elevated_skid_steer_drive'}">
+            <ode>
+              <mu>1</mu>
+              <mu2>1</mu2>
+              <slip1>0.015</slip1>
+              <slip2>0</slip2>
+              <fdir1>0 0 1</fdir1>
             </ode>
           </xacro:if>
@@ -543,4 +635,52 @@
       </plugin>
     </xacro:if>
+    <!-- controls big skid steer drive -->
+    <xacro:if value="${var == 'big_skid_steer_drive'}">
+      <plugin filename="gz-sim-diff-drive-system" name="gz::sim::systems::DiffDrive">
+        <left_joint>main_body_left_front_wheel</left_joint>
+        <left_joint>main_body_left_rear_wheel</left_joint>
+        <right_joint>main_body_right_front_wheel</right_joint>
+        <right_joint>main_body_right_rear_wheel</right_joint>
+        <wheel_separation>0.45</wheel_separation>
+        <wheel_radius>0.165</wheel_radius>
+        <max_linear_acceleration>5.5</max_linear_acceleration>
+        <min_linear_acceleration>-5.5</min_linear_acceleration>
+        <max_angular_acceleration>6</max_angular_acceleration>
+        <min_angular_acceleration>-6</min_angular_acceleration>
+        <max_linear_velocity>2.5</max_linear_velocity>
+        <min_linear_velocity>-2.5</min_linear_velocity>
+        <max_angular_velocity>3</max_angular_velocity>
+        <min_angular_velocity>-3</min_angular_velocity>
+        <topic>/robot/cmd_vel</topic>
+        <odom_topic>/robot/odom</odom_topic>
+        <tf_topic>/robot/tf</tf_topic>
+        <frame_id>odom</frame_id>
+        <child_frame_id>base_link</child_frame_id>
+      </plugin>
+    </xacro:if>
+    <!-- controls big skid steer drive -->
+    <xacro:if value="${var == 'elevated_skid_steer_drive'}">
+      <plugin filename="gz-sim-diff-drive-system" name="gz::sim::systems::DiffDrive">
+        <left_joint>main_body_left_front_wheel</left_joint>
+        <left_joint>main_body_left_rear_wheel</left_joint>
+        <right_joint>main_body_right_front_wheel</right_joint>
+        <right_joint>main_body_right_rear_wheel</right_joint>
+        <wheel_separation>0.45</wheel_separation>
+        <wheel_radius>0.165</wheel_radius>
+        <max_linear_acceleration>5.5</max_linear_acceleration>
+        <min_linear_acceleration>-5.5</min_linear_acceleration>
+        <max_angular_acceleration>6</max_angular_acceleration>
+        <min_angular_acceleration>-6</min_angular_acceleration>
+        <max_linear_velocity>2.5</max_linear_velocity>
+        <min_linear_velocity>-2.5</min_linear_velocity>
+        <max_angular_velocity>3</max_angular_velocity>
+        <min_angular_velocity>-3</min_angular_velocity>
+        <topic>/robot/cmd_vel</topic>
+        <odom_topic>/robot/odom</odom_topic>
+        <tf_topic>/robot/tf</tf_topic>
+        <frame_id>odom</frame_id>
+        <child_frame_id>base_link</child_frame_id>
+      </plugin>
+    </xacro:if>
     <!-- Controls the mecanum drive robot -->
     <xacro:if value="${var == 'mecanum_drive'}">
