Commit message: Update description package. This commit is auto-generated by the CI.

File: origin_one_description/urdf/origin_one.urdf.xacro (robot description, xacro)
@@ -1,5 +1,10 @@
 <?xml version='1.0'?>
-<robot name="avular_origin_one" xmlns:xacro="http://ros.org/wiki/xacro" xmlns:ignition="http://sdformat.org/schemas/root.xsd">
+<!-- Parametric description for the Avular Origin One. -->
+<robot name="avular_origin_one" xmlns:xacro="http://ros.org/wiki/xacro">
   <xacro:arg name="drive_configuration" default="skid_steer_drive"/>
+  <!-- Per-robot link/joint prefix (empty = none). -->
+  <xacro:arg name="prefix" default=""/>
+  <xacro:property name="prefix" value="$(arg prefix)"/>
+  <xacro:property name="P" value="${prefix + ('_' if prefix else '')}"/>
   <xacro:property name="var" value="$(arg drive_configuration)"/>
   <xacro:if value="${var == 'skid_steer_drive'}">
@@ -8,27 +13,13 @@
     <xacro:property name="wheelRadius" value="0.120"/>
     <xacro:property name="groundClearance" value="0.064"/>
-    <!-- wheelMeshFileA refer to the mesh file used to visualize front left & rear right wheel  -->
     <xacro:property name="wheelMeshFileA" value="package://origin_one_description/urdf/meshes/wheel.obj"/>
-    <!-- wheelMeshFileB refer to the mesh file used to visualize front right & rear left wheel  -->
     <xacro:property name="wheelMeshFileB" value="package://origin_one_description/urdf/meshes/wheel.obj"/>
   </xacro:if>
-  <xacro:if value="${var == 'big_skid_steer_drive'}">
+  <xacro:if value="${var == 'big_skid_steer_drive' or var == 'elevated_skid_steer_drive'}">
     <xacro:property name="trackWidth" value="0.530"/>
     <xacro:property name="wheelbase" value="0.410"/>
     <xacro:property name="wheelRadius" value="0.165"/>
     <xacro:property name="groundClearance" value="0.109"/>
-    <!-- wheelMeshFileA refer to the mesh file used to visualize front left & rear right wheel  -->
     <xacro:property name="wheelMeshFileA" value="package://origin_one_description/urdf/meshes/wheel_big.obj"/>
-    <!-- wheelMeshFileB refer to the mesh file used to visualize front right & rear left wheel  -->
-    <xacro:property name="wheelMeshFileB" value="package://origin_one_description/urdf/meshes/wheel_big.obj"/>
-  </xacro:if>
-  <xacro:if value="${var == 'elevated_skid_steer_drive'}">
-    <xacro:property name="trackWidth" value="0.530"/>
-    <xacro:property name="wheelbase" value="0.410"/>
-    <xacro:property name="wheelRadius" value="0.165"/>
-    <xacro:property name="groundClearance" value="0.109"/>
-    <!-- wheelMeshFileA refer to the mesh file used to visualize front left & rear right wheel  -->
-    <xacro:property name="wheelMeshFileA" value="package://origin_one_description/urdf/meshes/wheel_big.obj"/>
-    <!-- wheelMeshFileB refer to the mesh file used to visualize front right & rear left wheel  -->
     <xacro:property name="wheelMeshFileB" value="package://origin_one_description/urdf/meshes/wheel_big.obj"/>
   </xacro:if>
@@ -38,19 +29,49 @@
     <xacro:property name="wheelRadius" value="0.1015"/>
     <xacro:property name="groundClearance" value="0.0455"/>
-    <!-- wheelMeshFileA refer to the mesh file used to visualize front left & rear right wheel  -->
     <xacro:property name="wheelMeshFileA" value="package://origin_one_description/urdf/meshes/wheel_mecanumA.obj"/>
-    <!-- wheelMeshFileB refer to the mesh file used to visualize front right & rear left wheel  -->
     <xacro:property name="wheelMeshFileB" value="package://origin_one_description/urdf/meshes/wheel_mecanumB.obj"/>
   </xacro:if>
-  <gazebo>
-    <static>false</static>
-    <plugin filename="gz-sim-sensors-system" name="gz::sim::systems::Sensors">
-      <render_engine>ogre2</render_engine>
-    </plugin>
-    <plugin filename="ignition-gazebo-navsat-system" name="ignition::gazebo::systems::NavSat">
-    </plugin>
-  </gazebo>
-  <link name='base_link' />
-  <link name='main_body'>
+  <xacro:macro name="wheel_link" params="name visual_rpy mesh">
+    <link name="${P}${name}">
+      <inertial>
+        <mass value="1"/>
+        <inertia ixx="0.01" ixy="0.0" ixz="0.0" iyy="0.01" iyz="0.0" izz="0.01"/>
+      </inertial>
+      <collision>
+        <origin xyz="0 0 0.0" rpy="0 0 0"/>
+        <geometry>
+          <cylinder length=".07" radius="${wheelRadius}"/>
+        </geometry>
+      </collision>
+      <visual>
+        <origin xyz="0.0 0.0 0.0" rpy="${visual_rpy}"/>
+        <geometry>
+          <mesh filename="${mesh}"
+            scale="0.001 0.001 0.001" />
+        </geometry>
+      </visual>
+    </link>
+  </xacro:macro>
+  <xacro:macro name="wheel_joint" params="name xyz">
+    <joint type="continuous" name="${P}main_body_${name}">
+      <origin xyz="${xyz}" rpy="-1.5707 0 0"/>
+      <child link="${P}${name}" />
+      <parent link="${P}main_body"/>
+      <axis xyz="0 0 1"/>
+      <limit effort="100000.0" velocity="10"/>
+    </joint>
+  </xacro:macro>
+  <xacro:macro name="us_link" params="name">
+    <link name="${P}us_${name}_link"/>
+  </xacro:macro>
+  <xacro:macro name="us_joint" params="name xyz rpy">
+    <joint type="fixed" name="${P}us_${name}_joint">
+      <origin xyz="${xyz}" rpy="${rpy}"/>
+      <child link="${P}us_${name}_link"/>
+      <parent link="${P}main_body"/>
+    </joint>
+  </xacro:macro>
+  <link name='${P}base_link' />
+  <link name='${P}main_body'>
     <inertial>
       <mass value="21.0"/>
@@ -71,269 +92,9 @@
     </visual>
   </link>
-  <link name="left_front_wheel">
-    <inertial>
-      <mass value="1"/>
-      <inertia ixx="0.01" ixy="0.0" ixz="0.0" iyy="0.01" iyz="0.0" izz="0.01"/>
-    </inertial>
-    <collision>
-      <origin xyz="0 0 0.0" rpy="0 0 0"/>
-      <geometry>
-        <cylinder length=".07" radius="${wheelRadius}"/>
-      </geometry>
-    </collision>
-    <visual>
-      <origin xyz="0.0 0.0 0.0" rpy="0.0 1.5707 0.0"/>
-      <geometry>
-        <mesh filename="${wheelMeshFileA}"
-          scale="0.001 0.001 0.001" />
-      </geometry>
-    </visual>
-  </link>
-  <gazebo reference="left_front_wheel">
-    <collision>
-      <surface>
-        <friction>
-          <xacro:if value="${var == 'skid_steer_drive'}">
-            <ode>
-              <mu>1</mu>
-              <mu2>1</mu2>
-              <slip1>0.015</slip1>
-              <slip2>0</slip2>
-              <fdir1>0 0 1</fdir1>
-            </ode>
-          </xacro:if>
-          <xacro:if value="${var == 'mecanum_drive'}">
-            <ode>
-              <mu>1</mu>
-              <mu2>0</mu2>
-              <fdir1 ignition:expressed_in="base_link">1 -1 0</fdir1>
-            </ode>
-          </xacro:if>
-          <xacro:if value="${var == 'big_skid_steer_drive'}">
-            <ode>
-              <mu>1</mu>
-              <mu2>1</mu2>
-              <slip1>0.015</slip1>
-              <slip2>0</slip2>
-              <fdir1>0 0 1</fdir1>
-            </ode>
-          </xacro:if>
-          <xacro:if value="${var == 'elevated_skid_steer_drive'}">
-            <ode>
-              <mu>1</mu>
-              <mu2>1</mu2>
-              <slip1>0.015</slip1>
-              <slip2>0</slip2>
-              <fdir1>0 0 1</fdir1>
-            </ode>
-          </xacro:if>
-          <bullet>
-            <friction>1</friction>
-            <friction2>1</friction2>
-            <rolling_friction>0.1</rolling_friction>
-          </bullet>
-        </friction>
-      </surface>
-    </collision>
-  </gazebo>
-  <link name="right_front_wheel">
-    <inertial>
-      <mass value="1"/>
-      <inertia ixx="0.01" ixy="0.0" ixz="0.0" iyy="0.01" iyz="0.0" izz="0.01"/>
-    </inertial>
-    <collision>
-      <origin xyz="0 0 0.0" rpy="0 0 0"/>
-      <geometry>
-        <cylinder length=".07" radius="${wheelRadius}"/>
-      </geometry>
-    </collision>
-    <visual>
-      <origin xyz="0.0 0.0 0.0" rpy="0.0 -1.5707 0.0"/>
-      <geometry>
-        <mesh filename="${wheelMeshFileB}"
-          scale="0.001 0.001 0.001" />
-      </geometry>
-    </visual>
-  </link>
-  <gazebo reference="right_front_wheel">
-    <collision>
-      <surface>
-        <friction>
-          <xacro:if value="${var == 'skid_steer_drive'}">
-            <ode>
-              <mu>1</mu>
-              <mu2>1</mu2>
-              <slip1>0.015</slip1>
-              <slip2>0</slip2>
-              <fdir1>0 0 1</fdir1>
-            </ode>
-          </xacro:if>
-          <xacro:if value="${var == 'mecanum_drive'}">
-            <ode>
-              <mu>1</mu>
-              <mu2>0</mu2>
-              <fdir1 ignition:expressed_in="base_link">1 1 0</fdir1>
-            </ode>
-          </xacro:if>
-          <xacro:if value="${var == 'big_skid_steer_drive'}">
-            <ode>
-              <mu>1</mu>
-              <mu2>1</mu2>
-              <slip1>0.015</slip1>
-              <slip2>0</slip2>
-              <fdir1>0 0 1</fdir1>
-            </ode>
-          </xacro:if>
-          <xacro:if value="${var == 'elevated_skid_steer_drive'}">
-            <ode>
-              <mu>1</mu>
-              <mu2>1</mu2>
-              <slip1>0.015</slip1>
-              <slip2>0</slip2>
-              <fdir1>0 0 1</fdir1>
-            </ode>
-          </xacro:if>
-          <bullet>
-            <friction>1</friction>
-            <friction2>1</friction2>
-            <rolling_friction>0.1</rolling_friction>
-          </bullet>
-        </friction>
-      </surface>
-    </collision>
-  </gazebo>
-  <link name="left_rear_wheel">
-    <inertial>
-      <mass value="1"/>
-      <inertia ixx="0.01" ixy="0.0" ixz="0.0" iyy="0.01" iyz="0.0" izz="0.01"/>
-    </inertial>
-    <collision>
-      <origin xyz="0 0 0.0" rpy="0 0 0"/>
-      <geometry>
-        <cylinder length=".07" radius="${wheelRadius}"/>
-      </geometry>
-    </collision>
-    <visual>
-      <origin xyz="0.0 0.0 0.0" rpy="0.0 1.5707 0.0"/>
-      <geometry>
-        <mesh filename="${wheelMeshFileB}"
-          scale="0.001 0.001 0.001" />
-      </geometry>
-    </visual>
-  </link>
-  <gazebo reference="left_rear_wheel">
-    <collision>
-      <surface>
-        <friction>
-          <xacro:if value="${var == 'skid_steer_drive'}">
-            <ode>
-              <mu>1</mu>
-              <mu2>1</mu2>
-              <slip1>0.015</slip1>
-              <slip2>0</slip2>
-              <fdir1>0 0 1</fdir1>
-            </ode>
-          </xacro:if>
-          <xacro:if value="${var == 'mecanum_drive'}">
-            <ode>
-              <mu>1</mu>
-              <mu2>0</mu2>
-              <fdir1 ignition:expressed_in="base_link">1 1 0</fdir1>
-            </ode>
-          </xacro:if>
-          <xacro:if value="${var == 'big_skid_steer_drive'}">
-            <ode>
-              <mu>1</mu>
-              <mu2>1</mu2>
-              <slip1>0.015</slip1>
-              <slip2>0</slip2>
-              <fdir1>0 0 1</fdir1>
-            </ode>
-          </xacro:if>
-          <xacro:if value="${var == 'elevated_skid_steer_drive'}">
-            <ode>
-              <mu>1</mu>
-              <mu2>1</mu2>
-              <slip1>0.015</slip1>
-              <slip2>0</slip2>
-              <fdir1>0 0 1</fdir1>
-            </ode>
-          </xacro:if>
-          <bullet>
-            <friction>1</friction>
-            <friction2>1</friction2>
-            <rolling_friction>0.1</rolling_friction>
-          </bullet>
-        </friction>
-      </surface>
-    </collision>
-  </gazebo>
-  <link name="right_rear_wheel">
-    <inertial>
-      <mass value="1"/>
-      <inertia ixx="0.01" ixy="0.0" ixz="0.0" iyy="0.01" iyz="0.0" izz="0.01"/>
-    </inertial>
-    <collision>
-      <origin xyz="0 0 0.0" rpy="0 0 0"/>
-      <geometry>
-        <cylinder length=".07" radius="${wheelRadius}"/>
-      </geometry>
-    </collision>
-    <visual>
-      <origin xyz="0.0 0.0 0.0" rpy="0.0 -1.5707 0.0"/>
-      <geometry>
-        <mesh filename="${wheelMeshFileA}"
-          scale="0.001 0.001 0.001" />
-      </geometry>
-    </visual>
-  </link>
-  <gazebo reference="right_rear_wheel">
-    <collision>
-      <surface>
-        <friction>
-          <xacro:if value="${var == 'skid_steer_drive'}">
-            <ode>
-              <mu>1</mu>
-              <mu2>1</mu2>
-              <slip1>0.015</slip1>
-              <slip2>0</slip2>
-              <fdir1>0 0 1</fdir1>
-            </ode>
-          </xacro:if>
-          <xacro:if value="${var == 'mecanum_drive'}">
-            <ode>
-              <mu>1</mu>
-              <mu2>0</mu2>
-              <fdir1 ignition:expressed_in="base_link">1 -1 0</fdir1>
-            </ode>
-          </xacro:if>
-          <xacro:if value="${var == 'big_skid_steer_drive'}">
-            <ode>
-              <mu>1</mu>
-              <mu2>1</mu2>
-              <slip1>0.015</slip1>
-              <slip2>0</slip2>
-              <fdir1>0 0 1</fdir1>
-            </ode>
-          </xacro:if>
-          <xacro:if value="${var == 'elevated_skid_steer_drive'}">
-            <ode>
-              <mu>1</mu>
-              <mu2>1</mu2>
-              <slip1>0.015</slip1>
-              <slip2>0</slip2>
-              <fdir1>0 0 1</fdir1>
-            </ode>
-          </xacro:if>
-          <bullet>
-            <friction>1</friction>
-            <friction2>1</friction2>
-            <rolling_friction>0.1</rolling_friction>
-          </bullet>
-        </friction>
-      </surface>
-    </collision>
-  </gazebo>
-  <link name="ouster_base">
+  <xacro:wheel_link name="left_front_wheel"  visual_rpy="0.0 1.5707 0.0"  mesh="${wheelMeshFileA}"/>
+  <xacro:wheel_link name="right_front_wheel" visual_rpy="0.0 -1.5707 0.0" mesh="${wheelMeshFileB}"/>
+  <xacro:wheel_link name="left_rear_wheel"   visual_rpy="0.0 1.5707 0.0"  mesh="${wheelMeshFileB}"/>
+  <xacro:wheel_link name="right_rear_wheel"  visual_rpy="0.0 -1.5707 0.0" mesh="${wheelMeshFileA}"/>
+  <link name="${P}ouster_base">
     <inertial>
       <mass value="1"/>
@@ -353,52 +114,6 @@
     </collision>
   </link>
-  <link name="os_sensor" />
-  <link name="lidar_link_gazebo">
-    <inertial>
-      <mass value="0.1"/>
-      <inertia ixx="0.001" ixy="0.0" ixz="0.0" iyy="0.001" iyz="0.0" izz="0.001"/>
-    </inertial>
-    <collision name="collision-base">
-      <origin xyz="0 0 0.0" rpy="0 0 0"/>
-      <geometry>
-        <cylinder length="0.07" radius="0.04"/>
-      </geometry>
-    </collision>
-  </link>
-  <gazebo reference="lidar_link_gazebo">
-    <sensor name='ouster_lidar' type='gpu_lidar'>
-      <topic>/robot/lidar</topic>
-      <gz_frame_id>os_lidar</gz_frame_id>
-      <update_rate>10</update_rate>
-      <lidar>
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